File: water.sch (EAGLE design)
At the start: 15 parts, among them K1 AQH2223, K2 AQH2223, K3 AQH2223, K4 AQH2223, X5 MKDSN1,5/2-5,08, X6 MKDSN1,5/2-5,08, X7 MKDSN1,5/2-5,08, X8 MKDSN1,5/2-5,08

Commit message: Move parts
Parts:
- added SV2: (no value), con-lstb:MA04-2
- R1, R2, R3, R4: value 220 -> (none)
Connections:
- new net N$13: SV2.8, U2.CH_PD
- new net N$16: SV2.6, U2.RESET
- new net N$17: SV2.3, U2.TX
- new net N$18: SV2.1, U2.RX
- new net N$19: SV2.4, U2.GPIO15
- new net N$20: SV2.2, U2.GPIO0
- net +3V3: now also SV2.7
- net GND: now also SV2.5
Changed lines of the file:
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@@
 </classes>
 <parts>
-<part name="K1" library="relay" library_urn="urn:adsk.eagle:library:339" deviceset="AQH*223" device="" technology="2"/>
+<part name="K1" library="relay" library_urn="urn:adsk.eagle:library:339" deviceset="AQH*223" device="" technology="2" value="AQH2223"/>
 <part name="K2" library="relay" library_urn="urn:adsk.eagle:library:339" deviceset="AQH*223" device="" technology="2"/>
 <part name="K3" library="relay" library_urn="urn:adsk.eagle:library:339" deviceset="AQH*223" device="" technology="2"/>
@@
 <part name="X7" library="con-phoenix-508" library_urn="urn:adsk.eagle:library:176" deviceset="MKDSN1,5/2-5,08" device=""/>
 <part name="X8" library="con-phoenix-508" library_urn="urn:adsk.eagle:library:176" deviceset="MKDSN1,5/2-5,08" device=""/>
-<part name="R1" library="resistor" library_urn="urn:adsk.eagle:library:348" deviceset="R-EU_" device="R1206" value="220"/>
-<part name="R2" library="resistor" library_urn="urn:adsk.eagle:library:348" deviceset="R-EU_" device="R1206" value="220"/>
-<part name="R3" library="resistor" library_urn="urn:adsk.eagle:library:348" deviceset="R-EU_" device="R1206" value="220"/>
-<part name="R4" library="resistor" library_urn="urn:adsk.eagle:library:348" deviceset="R-EU_" device="R1206" value="220"/>
+<part name="R1" library="resistor" library_urn="urn:adsk.eagle:library:348" deviceset="R-EU_" device="R1206"/>
+<part name="R2" library="resistor" library_urn="urn:adsk.eagle:library:348" deviceset="R-EU_" device="R1206"/>
+<part name="R3" library="resistor" library_urn="urn:adsk.eagle:library:348" deviceset="R-EU_" device="R1206"/>
+<part name="R4" library="resistor" library_urn="urn:adsk.eagle:library:348" deviceset="R-EU_" device="R1206"/>
 <part name="GND1" library="supply1" library_urn="urn:adsk.eagle:library:371" deviceset="GND" device=""/>
 <part name="GND2" library="supply1" library_urn="urn:adsk.eagle:library:371" deviceset="GND" device=""/>
@@
 <part name="D1" library="diode" library_urn="urn:adsk.eagle:library:210" deviceset="1N4004" device=""/>
 <part name="GND7" library="supply1" library_urn="urn:adsk.eagle:library:371" deviceset="GND" device=""/>
+<part name="SV2" library="con-lstb" library_urn="urn:adsk.eagle:library:162" deviceset="MA04-2" device=""/>
+<part name="+3V3" library="supply1" library_urn="urn:adsk.eagle:library:371" deviceset="+3V3" device=""/>
+<part name="GND8" library="supply1" library_urn="urn:adsk.eagle:library:371" deviceset="GND" device=""/>
 </parts>
 <sheets>
@@
 <instance part="D1" gate="1" x="154.94" y="78.74"/>
 <instance part="GND7" gate="1" x="147.32" y="88.9"/>
+<instance part="SV2" gate="G$1" x="27.94" y="86.36"/>
+<instance part="+3V3" gate="G$1" x="43.18" y="93.98"/>
+<instance part="GND8" gate="1" x="48.26" y="83.82"/>
 </instances>
 <busses>
@@
 <wire x1="129.54" y1="91.44" x2="147.32" y2="91.44" width="0.1524" layer="91"/>
 </segment>
+<segment>
+<pinref part="SV2" gate="G$1" pin="5"/>
+<pinref part="GND8" gate="1" pin="GND"/>
+<wire x1="35.56" y1="86.36" x2="48.26" y2="86.36" width="0.1524" layer="91"/>
+</segment>
 </net>
 <net name="N$5" class="0">
@@
 <pinref part="+3V2" gate="G$1" pin="+3V3"/>
 <wire x1="17.78" y1="43.18" x2="5.08" y2="43.18" width="0.1524" layer="91"/>
+</segment>
+<segment>
+<pinref part="+3V3" gate="G$1" pin="+3V3"/>
+<pinref part="SV2" gate="G$1" pin="7"/>
+<wire x1="43.18" y1="91.44" x2="35.56" y2="91.44" width="0.1524" layer="91"/>
+<wire x1="35.56" y1="91.44" x2="35.56" y2="88.9" width="0.1524" layer="91"/>
 </segment>
 </net>
@@
 </segment>
 </net>
+<net name="N$13" class="0">
+<segment>
+<pinref part="SV2" gate="G$1" pin="8"/>
+<wire x1="20.32" y1="88.9" x2="12.7" y2="88.9" width="0.1524" layer="91"/>
+<wire x1="12.7" y1="88.9" x2="12.7" y2="55.88" width="0.1524" layer="91"/>
+<pinref part="U2" gate="G$1" pin="CH_PD"/>
+<wire x1="12.7" y1="55.88" x2="17.78" y2="55.88" width="0.1524" layer="91"/>
+</segment>
+</net>
+<net name="N$16" class="0">
+<segment>
+<pinref part="U2" gate="G$1" pin="RESET"/>
+<wire x1="17.78" y1="60.96" x2="15.24" y2="60.96" width="0.1524" layer="91"/>
+<wire x1="15.24" y1="60.96" x2="15.24" y2="86.36" width="0.1524" layer="91"/>
+<pinref part="SV2" gate="G$1" pin="6"/>
+<wire x1="15.24" y1="86.36" x2="20.32" y2="86.36" width="0.1524" layer="91"/>
+</segment>
+</net>
+<net name="N$17" class="0">
+<segment>
+<pinref part="U2" gate="G$1" pin="TX"/>
+<wire x1="50.8" y1="60.96" x2="50.8" y2="76.2" width="0.1524" layer="91"/>
+<wire x1="50.8" y1="76.2" x2="43.18" y2="76.2" width="0.1524" layer="91"/>
+<wire x1="43.18" y1="76.2" x2="43.18" y2="83.82" width="0.1524" layer="91"/>
+<pinref part="SV2" gate="G$1" pin="3"/>
+<wire x1="43.18" y1="83.82" x2="35.56" y2="83.82" width="0.1524" layer="91"/>
+</segment>
+</net>
+<net name="N$18" class="0">
+<segment>
+<pinref part="U2" gate="G$1" pin="RX"/>
+<wire x1="50.8" y1="58.42" x2="55.88" y2="58.42" width="0.1524" layer="91"/>
+<wire x1="55.88" y1="58.42" x2="55.88" y2="71.12" width="0.1524" layer="91"/>
+<pinref part="SV2" gate="G$1" pin="1"/>
+<wire x1="55.88" y1="71.12" x2="35.56" y2="71.12" width="0.1524" layer="91"/>
+<wire x1="35.56" y1="71.12" x2="35.56" y2="81.28" width="0.1524" layer="91"/>
+</segment>
+</net>
+<net name="N$19" class="0">
+<segment>
+<pinref part="SV2" gate="G$1" pin="4"/>
+<wire x1="20.32" y1="83.82" x2="17.78" y2="83.82" width="0.1524" layer="91"/>
+<wire x1="17.78" y1="83.82" x2="17.78" y2="66.04" width="0.1524" layer="91"/>
+<wire x1="17.78" y1="66.04" x2="38.1" y2="66.04" width="0.1524" layer="91"/>
+<wire x1="38.1" y1="66.04" x2="38.1" y2="45.72" width="0.1524" layer="91"/>
+<pinref part="U2" gate="G$1" pin="GPIO15"/>
+<wire x1="38.1" y1="45.72" x2="50.8" y2="45.72" width="0.1524" layer="91"/>
+</segment>
+</net>
+<net name="N$20" class="0">
+<segment>
+<pinref part="U2" gate="G$1" pin="GPIO0"/>
+<wire x1="50.8" y1="50.8" x2="40.64" y2="50.8" width="0.1524" layer="91"/>
+<wire x1="40.64" y1="50.8" x2="40.64" y2="68.58" width="0.1524" layer="91"/>
+<pinref part="SV2" gate="G$1" pin="2"/>
+<wire x1="40.64" y1="68.58" x2="20.32" y2="68.58" width="0.1524" layer="91"/>
+<wire x1="20.32" y1="68.58" x2="20.32" y2="81.28" width="0.1524" layer="91"/>
+</segment>
+</net>

Commit message: Add capacitors
Parts:
- added C1, C2: 470uf, resistor:CPOL-EUE5-10.5
Connections:
- new net N$21: K1.DS1, K2.DS1, K3.DS1, K4.DS1, X5-1.KL
- net +3V3: now also C1.+, C2.+
- net GND: now also C1.-, C2.-; no longer K1.DS1, K2.DS1, K3.DS1, K4.DS1, X5-1.KL

Commit message: Changes
Other:
- moved on the sheet: C1, C2
Changed lines of the file:
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@@
 <part name="C1" library="resistor" library_urn="urn:adsk.eagle:library:348" deviceset="CPOL-EU" device="E5-10.5" value="470uf"/>
 <part name="C2" library="resistor" library_urn="urn:adsk.eagle:library:348" deviceset="CPOL-EU" device="E5-10.5" value="470uf"/>
-<part name="+3V4" library="supply1" library_urn="urn:adsk.eagle:library:371" deviceset="+3V3" device=""/>
-<part name="GND7" library="supply1" library_urn="urn:adsk.eagle:library:371" deviceset="GND" device=""/>
 </parts>
 <sheets>
@@
 <instance part="U2" gate="G$1" x="35.56" y="53.34"/>
 <instance part="SV1" gate="G$1" x="185.42" y="81.28" rot="MR0"/>
-<instance part="GND5" gate="1" x="172.72" y="71.12"/>
-<instance part="+3V1" gate="G$1" x="172.72" y="91.44"/>
+<instance part="GND5" gate="1" x="160.02" y="86.36"/>
+<instance part="+3V1" gate="G$1" x="160.02" y="99.06"/>
 <instance part="+3V2" gate="G$1" x="5.08" y="45.72"/>
 <instance part="GND6" gate="1" x="55.88" y="40.64"/>
@@
 <instance part="+3V3" gate="G$1" x="43.18" y="93.98"/>
 <instance part="GND8" gate="1" x="48.26" y="83.82"/>
-<instance part="C1" gate="G$1" x="165.1" y="48.26"/>
-<instance part="C2" gate="G$1" x="175.26" y="48.26"/>
-<instance part="+3V4" gate="G$1" x="165.1" y="58.42"/>
-<instance part="GND7" gate="1" x="165.1" y="35.56"/>
+<instance part="C1" gate="G$1" x="160.02" y="93.98"/>
+<instance part="C2" gate="G$1" x="170.18" y="93.98"/>
 </instances>
 <busses>
@@
 </segment>
 <segment>
-<pinref part="SV1" gate="G$1" pin="2"/>
-<pinref part="GND5" gate="1" pin="GND"/>
-<wire x1="177.8" y1="81.28" x2="172.72" y2="81.28" width="0.1524" layer="91"/>
-<wire x1="172.72" y1="81.28" x2="172.72" y2="73.66" width="0.1524" layer="91"/>
-</segment>
-<segment>
 <pinref part="U2" gate="G$1" pin="GND"/>
 <pinref part="GND6" gate="1" pin="GND"/>
@@
 </segment>
 <segment>
+<pinref part="GND5" gate="1" pin="GND"/>
 <pinref part="C1" gate="G$1" pin="-"/>
 <pinref part="C2" gate="G$1" pin="-"/>
-<wire x1="165.1" y1="43.18" x2="175.26" y2="43.18" width="0.1524" layer="91"/>
-<pinref part="GND7" gate="1" pin="GND"/>
-<wire x1="165.1" y1="43.18" x2="165.1" y2="38.1" width="0.1524" layer="91"/>
-<junction x="165.1" y="43.18"/>
+<wire x1="160.02" y1="88.9" x2="170.18" y2="88.9" width="0.1524" layer="91"/>
+<junction x="160.02" y="88.9"/>
+<wire x1="170.18" y1="88.9" x2="170.18" y2="81.28" width="0.1524" layer="91"/>
+<junction x="170.18" y="88.9"/>
+<pinref part="SV1" gate="G$1" pin="2"/>
+<wire x1="170.18" y1="81.28" x2="177.8" y2="81.28" width="0.1524" layer="91"/>
 </segment>
 </net>
@@
 <net name="+3V3" class="0">
 <segment>
-<pinref part="+3V1" gate="G$1" pin="+3V3"/>
-<pinref part="SV1" gate="G$1" pin="3"/>
-<wire x1="172.72" y1="88.9" x2="177.8" y2="88.9" width="0.1524" layer="91"/>
-<wire x1="177.8" y1="88.9" x2="177.8" y2="83.82" width="0.1524" layer="91"/>
-</segment>
-<segment>
 <pinref part="U2" gate="G$1" pin="VCC"/>
 <pinref part="+3V2" gate="G$1" pin="+3V3"/>
@@
 </segment>
 <segment>
-<pinref part="+3V4" gate="G$1" pin="+3V3"/>
+<pinref part="+3V1" gate="G$1" pin="+3V3"/>
 <pinref part="C1" gate="G$1" pin="+"/>
-<wire x1="165.1" y1="55.88" x2="165.1" y2="50.8" width="0.1524" layer="91"/>
+<pinref part="SV1" gate="G$1" pin="3"/>
+<wire x1="177.8" y1="83.82" x2="177.8" y2="96.52" width="0.1524" layer="91"/>
 <pinref part="C2" gate="G$1" pin="+"/>
-<wire x1="165.1" y1="50.8" x2="175.26" y2="50.8" width="0.1524" layer="91"/>
-<junction x="165.1" y="50.8"/>
-</segment>
-</net>
+<wire x1="177.8" y1="96.52" x2="170.18" y2="96.52" width="0.1524" layer="91"/>
+<wire x1="170.18" y1="96.52" x2="160.02" y2="96.52" width="0.1524" layer="91"/>
+<junction x="170.18" y="96.52"/>
+<junction x="160.02" y="96.52"/>
+</segment>
+</net>

Commit message: Changes
Parts:
- added LED1, LED2, LED3: X42180, led:X42180
Changed lines of the file:
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@@
 <part name="C1" library="resistor" library_urn="urn:adsk.eagle:library:348" deviceset="CPOL-EU" device="E5-10.5" value="470uf"/>
 <part name="C2" library="resistor" library_urn="urn:adsk.eagle:library:348" deviceset="CPOL-EU" device="E5-10.5" value="470uf"/>
+<part name="LED1" library="led" library_urn="urn:adsk.eagle:library:259" deviceset="X42180" device=""/>
+<part name="LED2" library="led" library_urn="urn:adsk.eagle:library:259" deviceset="X42180" device=""/>
+<part name="LED3" library="led" library_urn="urn:adsk.eagle:library:259" deviceset="X42180" device=""/>
 </parts>
 <sheets>
@@
 <instance part="C1" gate="G$1" x="160.02" y="93.98"/>
 <instance part="C2" gate="G$1" x="170.18" y="93.98"/>
+<instance part="LED1" gate="G$1" x="185.42" y="30.48"/>
+<instance part="LED2" gate="G$1" x="205.74" y="30.48"/>
+<instance part="LED3" gate="G$1" x="226.06" y="30.48"/>
 </instances>
 <busses>

Commit message: Add led
Parts:
- removed LED2, LED3: X42180, led:X42180
- added R5: (no value), resistor:R-EU_R1206
Connections:
- new net N$22: LED1.A, R5.1
- net +3V3: now also R5.2
- net GND: now also LED1.C
Other:
- moved on the sheet: LED1
Changed lines of the file:
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@@
 <part name="C2" library="resistor" library_urn="urn:adsk.eagle:library:348" deviceset="CPOL-EU" device="E5-10.5" value="470uf"/>
 <part name="LED1" library="led" library_urn="urn:adsk.eagle:library:259" deviceset="X42180" device=""/>
-<part name="LED2" library="led" library_urn="urn:adsk.eagle:library:259" deviceset="X42180" device=""/>
-<part name="LED3" library="led" library_urn="urn:adsk.eagle:library:259" deviceset="X42180" device=""/>
+<part name="+3V4" library="supply1" library_urn="urn:adsk.eagle:library:371" deviceset="+3V3" device=""/>
+<part name="GND7" library="supply1" library_urn="urn:adsk.eagle:library:371" deviceset="GND" device=""/>
+<part name="R5" library="resistor" library_urn="urn:adsk.eagle:library:348" deviceset="R-EU_" device="R1206"/>
 </parts>
 <sheets>
@@
 <instance part="C1" gate="G$1" x="160.02" y="93.98"/>
 <instance part="C2" gate="G$1" x="170.18" y="93.98"/>
-<instance part="LED1" gate="G$1" x="185.42" y="30.48"/>
-<instance part="LED2" gate="G$1" x="205.74" y="30.48"/>
-<instance part="LED3" gate="G$1" x="226.06" y="30.48"/>
+<instance part="LED1" gate="G$1" x="172.72" y="48.26"/>
+<instance part="+3V4" gate="G$1" x="172.72" y="63.5"/>
+<instance part="GND7" gate="1" x="172.72" y="40.64"/>
+<instance part="R5" gate="G$1" x="172.72" y="55.88" rot="R90"/>
 </instances>
 <busses>
@@
 <wire x1="170.18" y1="81.28" x2="177.8" y2="81.28" width="0.1524" layer="91"/>
 </segment>
+<segment>
+<pinref part="LED1" gate="G$1" pin="C"/>
+<pinref part="GND7" gate="1" pin="GND"/>
+</segment>
 </net>
 <net name="N$5" class="0">
@@
 <junction x="170.18" y="96.52"/>
 <junction x="160.02" y="96.52"/>
+</segment>
+<segment>
+<pinref part="R5" gate="G$1" pin="2"/>
+<pinref part="+3V4" gate="G$1" pin="+3V3"/>
 </segment>
 </net>
@@
 </segment>
 </net>
+<net name="N$22" class="0">
+<segment>
+<pinref part="LED1" gate="G$1" pin="A"/>
+<pinref part="R5" gate="G$1" pin="1"/>
+</segment>
+</net>

Commit message: Add pogo test bed
Parts:
- removed LED1: X42180, led:X42180
- removed R5: (no value), resistor:R-EU_R1206
- added SV3, SV4: (no value), con-lstb:MA08-1
- added U1: (no value), my-parts:ESP12EPOGO
Connections:
- new net N$23: SV3.2, U1.GPIO13
- new net N$24: SV3.3, U1.GPIO12
- new net N$25: SV3.4, U1.GPIO14
- new net N$26: SV3.5, U1.GPIO16
- new net N$27: SV3.6, U1.CH_PD
- new net N$28: SV3.7, U1.ADC
- new net N$29: SV3.8, U1.RESET
- new net N$30: SV4.1, U1.GND
- new net N$31: SV4.2, U1.GPIO15
- new net N$32: SV4.3, U1.GPIO2
- new net N$33: SV4.4, U1.GPIO0
- new net N$34: SV4.5, U1.GPIO4
- new net N$35: SV4.6, U1.GPIO5
- new net N$36: SV4.7, U1.RX
- new net N$37: SV4.8, U1.TX
- net +3V3: no longer R5.2
- net GND: no longer LED1.C
- net N$22: now also SV3.1, U1.VCC; no longer LED1.A, R5.1
Changed lines of the file:
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@@
 <part name="C1" library="resistor" library_urn="urn:adsk.eagle:library:348" deviceset="CPOL-EU" device="E5-10.5" value="470uf"/>
 <part name="C2" library="resistor" library_urn="urn:adsk.eagle:library:348" deviceset="CPOL-EU" device="E5-10.5" value="470uf"/>
-<part name="LED1" library="led" library_urn="urn:adsk.eagle:library:259" deviceset="X42180" device=""/>
-<part name="+3V4" library="supply1" library_urn="urn:adsk.eagle:library:371" deviceset="+3V3" device=""/>
-<part name="GND7" library="supply1" library_urn="urn:adsk.eagle:library:371" deviceset="GND" device=""/>
-<part name="R5" library="resistor" library_urn="urn:adsk.eagle:library:348" deviceset="R-EU_" device="R1206"/>
+<part name="U1" library="my-parts" deviceset="ESP12E" device="POGO"/>
+<part name="SV3" library="con-lstb" library_urn="urn:adsk.eagle:library:162" deviceset="MA08-1" device=""/>
+<part name="SV4" library="con-lstb" library_urn="urn:adsk.eagle:library:162" deviceset="MA08-1" device=""/>
 </parts>
 <sheets>
@@
 <instance part="C1" gate="G$1" x="160.02" y="93.98"/>
 <instance part="C2" gate="G$1" x="170.18" y="93.98"/>
-<instance part="LED1" gate="G$1" x="172.72" y="48.26"/>
-<instance part="+3V4" gate="G$1" x="172.72" y="63.5"/>
-<instance part="GND7" gate="1" x="172.72" y="40.64"/>
-<instance part="R5" gate="G$1" x="172.72" y="55.88" rot="R90"/>
+<instance part="U1" gate="G$1" x="170.18" y="-12.7"/>
+<instance part="SV3" gate="1" x="144.78" y="-15.24"/>
+<instance part="SV4" gate="1" x="193.04" y="-15.24" rot="MR0"/>
 </instances>
 <busses>
@@
 <wire x1="170.18" y1="81.28" x2="177.8" y2="81.28" width="0.1524" layer="91"/>
 </segment>
-<segment>
-<pinref part="LED1" gate="G$1" pin="C"/>
-<pinref part="GND7" gate="1" pin="GND"/>
-</segment>
 </net>
 <net name="N$5" class="0">
@@
 <junction x="170.18" y="96.52"/>
 <junction x="160.02" y="96.52"/>
-</segment>
-<segment>
-<pinref part="R5" gate="G$1" pin="2"/>
-<pinref part="+3V4" gate="G$1" pin="+3V3"/>
 </segment>
 </net>
@@
 <net name="N$22" class="0">
 <segment>
-<pinref part="LED1" gate="G$1" pin="A"/>
-<pinref part="R5" gate="G$1" pin="1"/>
-</segment>
-</net>
+<pinref part="U1" gate="G$1" pin="VCC"/>
+<pinref part="SV3" gate="1" pin="1"/>
+</segment>
+</net>
+<net name="N$23" class="0">
+<segment>
+<pinref part="U1" gate="G$1" pin="GPIO13"/>
+<pinref part="SV3" gate="1" pin="2"/>
+</segment>
+</net>
+<net name="N$24" class="0">
+<segment>
+<pinref part="U1" gate="G$1" pin="GPIO12"/>
+<pinref part="SV3" gate="1" pin="3"/>
+</segment>
+</net>
+<net name="N$25" class="0">
+<segment>
+<pinref part="U1" gate="G$1" pin="GPIO14"/>
+<pinref part="SV3" gate="1" pin="4"/>
+</segment>
+</net>
+<net name="N$26" class="0">
+<segment>
+<pinref part="U1" gate="G$1" pin="GPIO16"/>
+<pinref part="SV3" gate="1" pin="5"/>
+</segment>
+</net>
+<net name="N$27" class="0">
+<segment>
+<pinref part="U1" gate="G$1" pin="CH_PD"/>
+<pinref part="SV3" gate="1" pin="6"/>
+</segment>
+</net>
+<net name="N$28" class="0">
+<segment>
+<pinref part="U1" gate="G$1" pin="ADC"/>
+<pinref part="SV3" gate="1" pin="7"/>
+</segment>
+</net>
+<net name="N$29" class="0">
+<segment>
+<pinref part="U1" gate="G$1" pin="RESET"/>
+<pinref part="SV3" gate="1" pin="8"/>
+</segment>
+</net>
+<net name="N$30" class="0">
+<segment>
+<pinref part="U1" gate="G$1" pin="GND"/>
+<pinref part="SV4" gate="1" pin="1"/>
+</segment>
+</net>
+<net name="N$31" class="0">
+<segment>
+<pinref part="U1" gate="G$1" pin="GPIO15"/>
+<pinref part="SV4" gate="1" pin="2"/>
+</segment>
+</net>
+<net name="N$32" class="0">
+<segment>
+<pinref part="U1" gate="G$1" pin="GPIO2"/>
+<pinref part="SV4" gate="1" pin="3"/>
+</segment>
+</net>
+<net name="N$33" class="0">
+<segment>
+<pinref part="U1" gate="G$1" pin="GPIO0"/>
+<pinref part="SV4" gate="1" pin="4"/>
+</segment>
+</net>
+<net name="N$34" class="0">
+<segment>
+<pinref part="U1" gate="G$1" pin="GPIO4"/>
+<pinref part="SV4" gate="1" pin="5"/>
+</segment>
+</net>
+<net name="N$35" class="0">
+<segment>
+<pinref part="U1" gate="G$1" pin="GPIO5"/>
+<pinref part="SV4" gate="1" pin="6"/>
+</segment>
+</net>
+<net name="N$36" class="0">
+<segment>
+<pinref part="U1" gate="G$1" pin="RX"/>
+<pinref part="SV4" gate="1" pin="7"/>
+</segment>
+</net>
+<net name="N$37" class="0">
+<segment>
+<pinref part="U1" gate="G$1" pin="TX"/>
+<pinref part="SV4" gate="1" pin="8"/>
+</segment>
+</net>
