File: water.brd (EAGLE design)
At the start: 50 x 50 mm, 22 parts, among them K1 AQH2223, K2 AQH2223, K3 AQH2223, K4 AQH2223, X5 MKDSN1,5/2-5,08, X6 MKDSN1,5/2-5,08, X7 MKDSN1,5/2-5,08, X8 MKDSN1,5/2-5,08

Commit message: Fix conflicts
Parts:
- removed D2: 1N4004, diode:DO41-10
- removed SV5: (no value), my-parts:DC-DC
- added SV1: (no value), con-lstb:MA03-1
- moved D1 6.00 mm to (41.6, 34.0)
- moved X7 1.00 mm to (31.0, 45.0)
- moved X8 1.00 mm to (43.0, 45.0)
Connections:
- net +3V3: now also SV1.3; no longer SV5.VO
- net GND: now also SV1.2; no longer D2.A, SV5.GND
- net N$14: now also SV1.1; no longer SV5.V1
- net N$21: no longer D2.C
Routing:
- net GND: track 141.6 -> 126.1 mm
- net N$14: track 17.0 -> 5.55 mm
- net N$21: track 120.0 -> 113.4 mm
- net +3V3: track 72.8 -> 66.7 mm
- net N$15: track 28.9 -> 34.9 mm
- net N$10: track 51.8 -> 51.0 mm
- net N$11: track 34.0 -> 33.2 mm
- net N$12: track 47.7 -> 47.0 mm
- net N$9: track 38.5 -> 37.8 mm

Commit message: revert to where it worked
Parts:
- removed SV1: (no value), con-lstb:MA03-1
- added D2: 1N4004, diode:DO41-10
- added SV5: (no value), my-parts:DC-DC
- moved D1 6.00 mm to (35.6, 34.0)
- moved X7 1.00 mm to (31.0, 46.0)
- moved X8 1.00 mm to (43.0, 46.0)
Connections:
- net +3V3: now also SV5.VO; no longer SV1.3
- net GND: now also D2.A, SV5.GND; no longer SV1.2
- net N$14: now also SV5.V1; no longer SV1.1
- net N$21: now also D2.C
Routing:
- net GND: track 126.1 -> 141.6 mm
- net N$14: track 5.55 -> 17.0 mm
- net N$21: track 113.4 -> 120.0 mm
- net +3V3: track 66.7 -> 72.8 mm
- net N$15: track 34.9 -> 28.9 mm
- net N$10: track 51.0 -> 51.8 mm
- net N$11: track 33.2 -> 34.0 mm
- net N$12: track 47.0 -> 47.7 mm
- net N$9: track 37.8 -> 38.5 mm
